File: hardware/epaper-breakout/epaper-breakout.sch (KiCad schematic (older format))
At the start: 90 parts, among them J1 XF2M-3315-1A, J2 C10418, J3 Conn_02x06_Counter_Clockwise, J4 ED060SC4, J5 Conn_01x01_Male, J6 Conn_01x01_Male, Q1 AO3401A, Q2 AO3401A, Q3 MMBT3904, Q4 MMBT3904, Q5 AO3401A, Q6 MMBT3904, U1 MCP1700-3302E_SOT23, U10 ED060SC7, U11 TP4056, U12 CH340C, U2 LT1945, U3 LT1945, U4 XC6206PxxxMR, U5 ESP32-WROVER, U6 ED060XC5, U7 LM358, U8 74HC4094-normal, U9 MCP9700AT-ETT

Commit message: first schematic based on tps65185
Parts:
- removed C1, C6: 4.7uF, Capacitor_SMD:C_0603_1608Metric, symbol Device:CP
- removed JP_TEMP1: Jumper, Jumper:SolderJumper-2_P1.3mm_Bridged2Bar_RoundedPad1.0x1.5mm, symbol Device:Jumper
- removed L3, L4: 22uH, Inductor_SMD:L_6.3x6.3_H3, symbol Device:L
- removed Q2, Q5: AO3401A, Package_TO_SOT_SMD:SOT-23, symbol Transistor_FET:AO3401A
- removed Q6: MMBT3904, Package_TO_SOT_SMD:SOT-23, symbol Transistor_BJT:MMBT3904
- removed RV1: 200k, epaper-breakout:EVM3ESX50B25, symbol Device:R_POT
- removed TP1: TestPoint_Probe, TestPoint:TestPoint_Pad_D1.0mm, symbol Connector:TestPoint_Probe
- removed U2, U3: LT1945, Package_SO:MSOP-10_3x3mm_P0.5mm, symbol Regulator_Switching:LT1945
- removed U7: LM358, Package_SO:SOP-8_3.76x4.96mm_P1.27mm, symbol Amplifier_Operational:LM358
- removed U8: 74HC4094-normal, Package_SO:SOIC-16_3.9x9.9mm_P1.27mm, symbol 74HC4094:74HC4094-normal
- removed U9: MCP9700AT-ETT, Package_TO_SOT_SMD:SOT-23, symbol Sensor_Temperature:MCP9700AT-ETT
- added C1, C24, C26, C28, C31: 4.7uF, Capacitor_SMD:C_0603_1608Metric, symbol Device:C
- added C25: 10nF, Capacitor_SMD:C_0603_1608Metric, symbol Device:C
- added C27, C33: 2.2uF, Capacitor_SMD:C_0603_1608Metric, symbol Device:C
- added C29, C30: 100nF, Capacitor_SMD:C_0603_1608Metric, symbol Device:C
- added C32: 10uF, Capacitor_SMD:C_0603_1608Metric, symbol Device:C
- added C6: 47uF, Capacitor_SMD:C_0603_1608Metric, symbol Device:C
- added J7: Conn_01x10, symbol Connector_Generic:Conn_01x10
- added R23: 1M, Resistor_SMD:R_0805_2012Metric, symbol Device:R
- added R24: 47.5k, Resistor_SMD:R_0805_2012Metric, symbol Device:R
- added R25: 10k, Resistor_SMD:R_0805_2012Metric, symbol Device:R
- added TH1: 100k, symbol Device:Thermistor_NTC
- added U2: PCA9555PW, Package_SO:TSSOP-24_4.4x7.8mm_P0.65mm, symbol Interface_Expansion:PCA9555PW
- added U3: TPS651851RSLR, RSL48_4P4X4P4, symbol TPS651851RSLR:TPS651851RSLR
- C10: value 4.7pF -> 47uF; LCSC C1669 -> C19702
- C11, C8: value 100pF -> 4.7uF; LCSC C14858 -> C19702
- C12, C19, C9: value 1uF -> 10uF; LCSC C15849 -> C19702
- C20: value 1uF -> 10nF; LCSC C15849 -> C14858
- C4, C7: value 0.1uF -> 4.7uF; LCSC C14663 -> C19702
- C5: value 4.7pF -> 4.7uF; LCSC C1669 -> C19702
- L1: value 22uH -> 4.7uH
- L2: value 22uH -> 2.2uH; LCSC C206321 -> C206321
- R12: value 1k -> 0; footprint Resistor_SMD:R_0805_2012Metric -> (none); LCSC C17513 -> (none)
- R14: value 390k -> 10k; LCSC C17656 -> C17414
- R16: value 300k -> 10k; LCSC C17616 -> C17414
- R17: value 27k -> 1M; LCSC C17593 -> C17616
- R18: value 110k -> 43k; footprint Resistor_SMD:R_0805_2012Metric -> (none); LCSC C17422 -> (none)
- R19: value 10k -> 1M; LCSC C17414 -> C17616
- R20: value 10k -> 52.3k; LCSC C17414 -> C17593
- R4: value 2M -> 10k; LCSC C26112 -> C17414
- R5: value 120k -> 0; footprint Resistor_SMD:R_0805_2012Metric -> (none); LCSC C17436 -> (none)
- R6: value 560k -> 10k; LCSC C15785 -> C17414
- R7: value 39k -> 0; footprint Resistor_SMD:R_0805_2012Metric -> (none); LCSC C25826 -> (none)
Connections:
- net labels added: SCL, SDA, TPS_PWRUP, TPS_PWR_GOOD, TPS_VCOM_CTRL, TPS_WAKEUP, TPS_nINT, VNEG_IN, ~GPIO_INTR
- net labels removed: A1, CTRL+15V, CTRL+22V, CTRL-15V, CTRL-20V, SMPS_CTRL, V_TEMP
- wire segments 498 -> 509
- no-connect marks 28 -> 31
Other:
- note removed: "Epaper Common Voltage"
- note removed: "SMPS Power +22V, -20V"
- note removed: "Unused opamp neutralizer"
- moved on the sheet: C13, C14, C15, C16, C17, C18, C2, C21, C22, C23, C3, D10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
